File: High Power SW.sch (KiCad schematic (older format))
At the start: 15 parts, among them CN1 Jumper_NC_Small, Q1 PSMN5R6-60YLX, U1 TLP182

Commit message: Update opto footprint and add logos
Parts:
- FAN: Supplier (none) -> Digi-Key; Supplier_Part_No (none) -> None
- U1: footprint MyLib:SOP-4 -> MyLib:OP_Hybrid; symbol TLP290 -> TLP182
Connections:
- net +BATT: now also U1.6; no longer U1.4
- net at JP1.1, R4.2: now also U1.3; no longer U1.2
- net at R1.1: now also U1.4; no longer U1.3
Changed lines of the file:
@@
 $EndComp
 $Comp
-L +BATT #PWR01
+L +BATT #PWR8
 U 1 1 580AECD6
 P 7200 4300
-F 0 "#PWR01" H 7200 4150 50  0001 C CNN
+F 0 "#PWR8" H 7200 4150 50  0001 C CNN
 F 1 "+BATT" H 7200 4440 50  0000 C CNN
 F 2 "" H 7200 4300 50  0000 C CNN
@@
 $EndComp
 $Comp
-L TLP290 U1
+L TLP182 U1
 U 1 1 581E947F
 P 5450 4350
 F 0 "U1" H 5275 4125 50  0000 L CNN
 F 1 "TLP182" H 5325 4575 50  0000 L CNN
-F 2 "MyLib:SOP-4" H 5250 4150 50  0001 L CIN
+F 2 "MyLib:OP_Hybrid" H 5250 4150 50  0001 L CIN
 F 3 "https://toshiba.semicon-storage.com/info/docget.jsp?did=14414&prodName=TLP182" H 5450 4350 50  0001 L CNN
 F 4 "Digi-Key" H 5450 4350 60  0001 C CNN "Supplier"
@@
 $EndComp
 $Comp
-L +BATT #PWR02
+L +BATT #PWR3
 U 1 1 581EA16D
 P 5775 4000
-F 0 "#PWR02" H 5775 3850 50  0001 C CNN
+F 0 "#PWR3" H 5775 3850 50  0001 C CNN
 F 1 "+BATT" H 5775 4140 50  0000 C CNN
 F 2 "" H 5775 4000 50  0000 C CNN
@@
 F 2 "MyLib:6pin_SMT_HEADER" H 3500 4975 50  0001 C CNN
 F 3 "-NA-" H 3500 4975 50  0001 C CNN
-F 4 "-NA-" H 3500 4975 60  0001 C CNN "mfr_num"
-F 5 "-NA-" H 3500 4975 60  0001 C CNN "Manufacturer"
-F 6 "-NA-" H 3500 4975 60  0001 C CNN "Supplyer"
-F 7 "-NA-" H 3500 4975 60  0001 C CNN "Supplyer_Link"
-F 8 "-NA-" H 3500 4975 60  0001 C CNN "Supplyer_Part_No"
-F 9 "-NA-" H 3500 4975 60  0001 C CNN "Reel_Part_No"
-F 10 "-NA-" H 3500 4975 60  0001 C CNN "Parts_Per_Reel"
+F 4 "Digi-Key" H 3500 4975 60  0001 C CNN "Supplier"
+F 5 "None" H 3500 4975 60  0001 C CNN "Supplier_Part_No"
+F 6 "-NA-" H 3500 4975 60  0001 C CNN "Manufacturer"
+F 7 "-NA-" H 3500 4975 60  0001 C CNN "mfr_num"
+F 8 "-NA-" H 3500 4975 60  0001 C CNN "Supplyer"
+F 9 "-NA-" H 3500 4975 60  0001 C CNN "Supplyer_Link"
+F 10 "-NA-" H 3500 4975 60  0001 C CNN "Supplyer_Part_No"
+F 11 "-NA-" H 3500 4975 60  0001 C CNN "Reel_Part_No"
+F 12 "-NA-" H 3500 4975 60  0001 C CNN "Parts_Per_Reel"
 	1    3500 4975
 	-1   0    0    -1
 $EndComp
 $Comp
-L +BATT #PWR03
+L +BATT #PWR1
 U 1 1 58410D16
 P 3700 4825
-F 0 "#PWR03" H 3700 4675 50  0001 C CNN
+F 0 "#PWR1" H 3700 4675 50  0001 C CNN
 F 1 "+BATT" H 3700 4965 50  0000 C CNN
 F 2 "" H 3700 4825 50  0000 C CNN
@@
 $EndComp
 $Comp
-L GND #PWR04
+L GND #PWR2
 U 1 1 58410D9F
 P 3700 5125
-F 0 "#PWR04" H 3700 4875 50  0001 C CNN
+F 0 "#PWR2" H 3700 4875 50  0001 C CNN
 F 1 "GND" H 3700 4975 50  0000 C CNN
 F 2 "" H 3700 5125 50  0000 C CNN
@@
 $EndComp
 $Comp
-L GND #PWR05
+L GND #PWR6
 U 1 1 584239D3
 P 6375 5225
-F 0 "#PWR05" H 6375 4975 50  0001 C CNN
+F 0 "#PWR6" H 6375 4975 50  0001 C CNN
 F 1 "GND" H 6375 5075 50  0000 C CNN
 F 2 "" H 6375 5225 50  0000 C CNN
@@
 $EndComp
 $Comp
-L +BATT #PWR06
+L +BATT #PWR5
 U 1 1 58423EEF
 P 6375 4000
-F 0 "#PWR06" H 6375 3850 50  0001 C CNN
+F 0 "#PWR5" H 6375 3850 50  0001 C CNN
 F 1 "+BATT" H 6375 4140 50  0000 C CNN
 F 2 "" H 6375 4000 50  0000 C CNN
@@
 $EndComp
 $Comp
-L GND #PWR07
+L GND #PWR4
 U 1 1 5842462A
 P 5775 5225
-F 0 "#PWR07" H 5775 4975 50  0001 C CNN
+F 0 "#PWR4" H 5775 4975 50  0001 C CNN
 F 1 "GND" H 5775 5075 50  0000 C CNN
 F 2 "" H 5775 5225 50  0000 C CNN
@@
 $EndComp
 $Comp
-L GND #PWR08
+L GND #PWR7
 U 1 1 580AECBB
 P 7050 4400
-F 0 "#PWR08" H 7050 4150 50  0001 C CNN
+F 0 "#PWR7" H 7050 4150 50  0001 C CNN
 F 1 "GND" H 7050 4250 50  0000 C CNN
 F 2 "" H 7050 4400 50  0000 C CNN

Commit message: Updated bill of materials
Parts:
- BED+, BED-, POWER+, POWER-: Parts_Per_Reel NA -> (none); Reel_Part_No NA -> (none)
- CN1: Parts_Per_Reel 6600 -> (none)
- D3: Parts_Per_Reel 2500 -> (none); Reel_Part_No CLM1B-AKW-CUAVB253TR-ND -> (none)
- FAN: Parts_Per_Reel -NA- -> (none); Reel_Part_No -NA- -> (none); Supplier Digi-Key -> (none); Supplier_Part_No None -> (none)
- Q1: Parts_Per_Reel 1500 -> (none); Reel_Part_No 568-13047-2-ND -> (none); Supplier Digi-Key -> (none); Supplier_Part_No None -> (none)
- R1: Cost .1 -> (none); Parts_Per_Reel 5000 -> (none); Reel_Part_No 311-1.00KFRTR-ND -> (none)
- R2: Cost .1 -> (none); Parts_Per_Reel 5000 -> (none); Reel_Part_No 311-1.80FRTR-ND -> (none)
- R3: Supplier Digi-Key -> (none); Supplier_Part_No None -> (none)
- R4: Cost .1 -> (none); Parts_Per_Reel 5000 -> (none); Reel_Part_No 311-1.69KFRTR-ND -> (none)
- R5: Parts_Per_Reel 5000 -> (none); Reel_Part_No 311-3.60FRTR-ND -> (none)
- U1: Parts_Per_Reel 3000 -> (none); Reel_Part_No TLP182(BL-TPLETR-ND -> (none); Supplier Digi-Key -> (none); Supplier_Part_No None -> (none)
Other:
- moved on the sheet: BED+, BED-, CN1, D3, FAN, JP1, POWER+, POWER-, Q1, R1, R2, R3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

Commit message: Update Board Design based on feedback
Parts:
- BED+, BED-, POWER+, POWER-: Parts_Per_Reel (none) -> NA; Reel_Part_No (none) -> NA
- CN1: Parts_Per_Reel (none) -> 6600
- D3: Parts_Per_Reel (none) -> 2500; Reel_Part_No (none) -> CLM1B-AKW-CUAVB253TR-ND
- FAN: Parts_Per_Reel (none) -> -NA-; Reel_Part_No (none) -> -NA-
- Q1: Parts_Per_Reel (none) -> 1500; Reel_Part_No (none) -> 568-13047-2-ND
- R1: Cost (none) -> .1; Parts_Per_Reel (none) -> 5000; Reel_Part_No (none) -> 311-1.00KFRTR-ND
- R2: Cost (none) -> .1; Parts_Per_Reel (none) -> 5000; Reel_Part_No (none) -> 311-1.80FRTR-ND
- R3: Cost (none) -> .1; Parts_Per_Reel (none) -> 5000; Reel_Part_No (none) -> 311-300ERTR-ND
- R4: Cost (none) -> .1; Parts_Per_Reel (none) -> 5000; Reel_Part_No (none) -> 311-1.69KFRTR-ND
- R5: Parts_Per_Reel (none) -> 5000; Reel_Part_No (none) -> 311-3.60FRTR-ND
- U1: value TLP182 -> PS2801C-1-A; footprint MyLib:OP_Hybrid -> MyLib:SOP-4; symbol TLP182 -> LTV-356T; Manufacturer Toshiba Semiconductor and Storage -> CEL; Parts_Per_Reel (none) -> 3500; Reel_Part_No (none) -> PS2801C-1-F3-ATR-ND; Supplyer_Link https://www.digikey.com/product-detail/en/toshiba-semicondu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 -> http://www.digikey.com/product-search/en?keywords=PS2801C-1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; Supplyer_Part_No TLP182(BL-TPLECT-ND -> PS2801C-1-A-ND; mfr_num TLP182(BL-TPL,E -> PS2801C-1-A
Other:
- note added: "Power - 11v - 30v\nJP1 - Install if input trigger is between 3.0v - 5.5v\nJP1 - Remote if input trigger is between 10v - 30v\n\nThe input trigger is opticly isolated from the bed power supply.\n\n30A Max curent through bed terminals. Q1 is capable of 100A \nat 25 deg C but the power terminals are rated for 30A per pin.\n\nMax size heated bed\n 30v - 900Watts (1.0 Ohms)\n 24v - 720Watts (0.8 Ohms)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"
- note removed: "Power - 10v - 30v\nJP1 - Install if input trigger is between 2.8v - 15v, 15v is the Absolut Max\nJP1 - Remote if input trigger is between 10v - 30v, 30v is the Absolut Max\n\nThe input trigger is opticly isolated from the bed power supply.\n\n30A Max curent through bed terminals. Q1 is capable of 100A \nat 25 deg C but the power terminals are rated for 30A per pin.\n\nMax size heated bed\n 30v - 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"
- moved on the sheet: BED+, BED-, CN1, D3, FAN, JP1, POWER+, POWER-, Q1, R1, R2, R3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

Commit message: Compleat Redesign
Parts:
- Q1: value PSMN5R6-60YLX -> IRFR7540TRPBF; footprint TO_SOT_Packages_SMD:SOT-669_LFPAK_ThermalVias-2 -> MyLib:TO-263-2Lead_(Small_Heat_Sink); symbol PSMN5R6-60YLX -> Q_NMOS_GDSD; Manufacturer Nexperia USA Inc. -> Infineon Technologies; Parts_Per_Reel 1500 -> (none); Reel_Part_No 568-13047-2-ND -> (none); Supplyer_Part_No 568-13047-1-ND -> IRFR7540TRPBFCT-ND; mfr_num PSMN5R6-60YLX -> IRFR7540TRPBF
- U1: footprint MyLib:SOP-4 -> MyLib:OP_Hybrid; symbol LTV-356T -> TLP182
Connections:
- net GND: no longer Q1.1 (S), Q1.2 (S)
- net at R1.2, R2.1: now also Q1.1 (G); no longer Q1.4 (G)
- net at BED-.1 (P1), D3.1 (K): now also Q1.2 (D), Q1.4 (D); no longer Q1.5 (D)
Changed lines of the file:
@@
 $EndComp
 $Comp
-L +BATT #PWR01
+L +BATT #PWR8
 U 1 1 580AECD6
 P 4525 2350
-F 0 "#PWR01" H 4525 2200 50  0001 C CNN
+F 0 "#PWR8" H 4525 2200 50  0001 C CNN
 F 1 "+BATT" H 4525 2490 50  0000 C CNN
 F 2 "" H 4525 2350 50  0000 C CNN
@@
 $EndComp
 $Comp
-L LTV-356T U1
+L TLP182 U1
 U 1 1 581E947F
 P 2775 2400
 F 0 "U1" H 2600 2175 50  0000 L CNN
 F 1 "PS2801C-1-A" H 2425 2600 50  0000 L CNN
-F 2 "MyLib:SOP-4" H 2575 2200 50  0001 L CIN
+F 2 "MyLib:OP_Hybrid" H 2575 2200 50  0001 L CIN
 F 3 "http://www.cel.com/pdf/datasheets/PS2801C-1,PS2801C-4.pdf" H 2775 2400 50  0001 L CNN
 F 4 "PS2801C-1-A" H 2775 2400 60  0001 C CNN "mfr_num"
@@
 $EndComp
 $Comp
-L +BATT #PWR02
+L +BATT #PWR3
 U 1 1 581EA16D
 P 3100 2050
-F 0 "#PWR02" H 3100 1900 50  0001 C CNN
+F 0 "#PWR3" H 3100 1900 50  0001 C CNN
 F 1 "+BATT" H 3100 2190 50  0000 C CNN
 F 2 "" H 3100 2050 50  0000 C CNN
@@
 $EndComp
 $Comp
-L +BATT #PWR03
+L +BATT #PWR1
 U 1 1 58410D16
 P 1025 2875
-F 0 "#PWR03" H 1025 2725 50  0001 C CNN
+F 0 "#PWR1" H 1025 2725 50  0001 C CNN
 F 1 "+BATT" H 1025 3015 50  0000 C CNN
 F 2 "" H 1025 2875 50  0000 C CNN
@@
 $EndComp
 $Comp
-L GND #PWR04
+L GND #PWR2
 U 1 1 58410D9F
 P 1025 3175
-F 0 "#PWR04" H 1025 2925 50  0001 C CNN
+F 0 "#PWR2" H 1025 2925 50  0001 C CNN
 F 1 "GND" H 1025 3025 50  0000 C CNN
 F 2 "" H 1025 3175 50  0000 C CNN
@@
 $EndComp
 $Comp
-L GND #PWR05
+L GND #PWR6
 U 1 1 584239D3
 P 3700 3275
-F 0 "#PWR05" H 3700 3025 50  0001 C CNN
+F 0 "#PWR6" H 3700 3025 50  0001 C CNN
 F 1 "GND" H 3700 3125 50  0000 C CNN
 F 2 "" H 3700 3275 50  0000 C CNN
@@
 $EndComp
 $Comp
-L +BATT #PWR06
+L +BATT #PWR5
 U 1 1 58423EEF
 P 3700 2050
-F 0 "#PWR06" H 3700 1900 50  0001 C CNN
+F 0 "#PWR5" H 3700 1900 50  0001 C CNN
 F 1 "+BATT" H 3700 2190 50  0000 C CNN
 F 2 "" H 3700 2050 50  0000 C CNN
@@
 $EndComp
 $Comp
-L GND #PWR07
+L GND #PWR4
 U 1 1 5842462A
 P 3100 3275
-F 0 "#PWR07" H 3100 3025 50  0001 C CNN
+F 0 "#PWR4" H 3100 3025 50  0001 C CNN
 F 1 "GND" H 3100 3125 50  0000 C CNN
 F 2 "" H 3100 3275 50  0000 C CNN
@@
 $EndComp
 $Comp
-L GND #PWR08
+L GND #PWR7
 U 1 1 580AECBB
 P 4375 2450
-F 0 "#PWR08" H 4375 2200 50  0001 C CNN
+F 0 "#PWR7" H 4375 2200 50  0001 C CNN
 F 1 "GND" H 4375 2300 50  0000 C CNN
 F 2 "" H 4375 2450 50  0000 C CNN
@@
 Connection ~ 4525 2500
 Wire Wire Line
-	3700 3125 3700 3275
-Wire Wire Line
 	3700 2050 3700 2100
 Wire Wire Line
@@
 Little Driver is licensed under a\nCreative Commons Attribution-ShareAlike 3.0 Unported License.
 $Comp
-L PSMN5R6-60YLX Q1
+L Q_NMOS_GDSD Q1
 U 1 1 58A00EB2
 P 3600 2925
 F 0 "Q1" H 3800 2975 50  0000 L CNN
-F 1 "PSMN5R6-60YLX" H 3800 2875 50  0000 L CNN
-F 2 "TO_SOT_Packages_SMD:SOT-669_LFPAK_ThermalVias-2" H 3800 3025 50  0001 C CNN
-F 3 "http://cache.nxp.com/documents/data_sheet/PSMN5R6-60YL.pdf" H 3600 2925 50  0001 C CNN
-F 4 "PSMN5R6-60YLX" H 3600 2925 60  0001 C CNN "mfr_num"
-F 5 "Nexperia USA Inc." H 3600 2925 60  0001 C CNN "Manufacturer"
+F 1 "IRFR7540TRPBF" H 3800 2875 50  0000 L CNN
+F 2 "MyLib:TO-263-2Lead_(Small_Heat_Sink)" H 3800 3025 50  0001 C CNN
+F 3 "http://www.infineon.com/dgdl/irfr7540pbf.pdf?fileId=5546d462533600a401535635b06a211c" H 3600 2925 50  0001 C CNN
+F 4 "IRFR7540TRPBF" H 3600 2925 60  0001 C CNN "mfr_num"
+F 5 "Infineon Technologies" H 3600 2925 60  0001 C CNN "Manufacturer"
 F 6 "Digi-Key" H 3600 2925 60  0001 C CNN "Supplyer"
 F 7 "http://www.digikey.com/product-detail/en/nexperia-usa-inc/PSMN5R6-60YLX/568-13047-1-ND/6167607" H 3600 2925 60  0001 C CNN "Supplyer_Link"
-F 8 "568-13047-1-ND" H 3600 2925 60  0001 C CNN "Supplyer_Part_No"
-F 9 "568-13047-2-ND" H 3600 2925 60  0001 C CNN "Reel_Part_No"
-F 10 "1500" H 3600 2925 60  0001 C CNN "Parts_Per_Reel"
+F 8 "IRFR7540TRPBFCT-ND" H 3600 2925 60  0001 C CNN "Supplyer_Part_No"
 	1    3600 2925
 	1    0    0    -1
@@
 	3700 2400 3700 2450
 Connection ~ 3700 2700
-Wire Wire Line
-	3800 3200 3800 3125
-Wire Wire Line
-	3900 3200 3900 3125
-Wire Wire Line
-	3700 3200 3900 3200
-Connection ~ 3800 3200
-Connection ~ 3700 3200
 $Comp
 L CONN_01X01 POWER+
@@
 	1    0    0    -1
 $EndComp
+Wire Wire Line
+	3700 3125 3700 3275
+Wire Wire Line
+	3800 2725 3800 2700
+Connection ~ 3800 2700
 $EndSCHEMATC

Commit message: Fixed issues with manufacture
Parts:
- BED+, BED-, POWER+, POWER-: Parts_Per_Reel NA -> (none); Reel_Part_No NA -> (none)
- CN1: Parts_Per_Reel 6600 -> (none)
- D3: Parts_Per_Reel 2500 -> (none); Reel_Part_No CLM1B-AKW-CUAVB253TR-ND -> (none)
- FAN: Parts_Per_Reel -NA- -> (none); Reel_Part_No -NA- -> (none)
- JP1: Parts_Per_Reel None -> (none); Reel_Part_No None -> (none)
- R1: Cost .1 -> (none); Parts_Per_Reel 5000 -> (none); Reel_Part_No 311-1.00KFRTR-ND -> (none)
- R2: Cost .1 -> (none); Parts_Per_Reel 5000 -> (none); Reel_Part_No 311-1.80FRTR-ND -> (none)
- R3: Cost .1 -> (none); Parts_Per_Reel 5000 -> (none); Reel_Part_No 311-300ERTR-ND -> (none)
- R4: Cost .1 -> (none); Parts_Per_Reel 5000 -> (none); Reel_Part_No 311-1.69KFRTR-ND -> (none)
- R5: Parts_Per_Reel 5000 -> (none); Reel_Part_No 311-3.60FRTR-ND -> (none)
- U1: Parts_Per_Reel 3500 -> (none); Reel_Part_No PS2801C-1-F3-ATR-ND -> (none)
Changed lines of the file:
@@
 F 7 "http://www.digikey.com/product-detail/en/yageo/RC1206FR-071KL/311-1.00KFRCT-ND/731334" H 1850 2500 60  0001 C CNN "Supplyer_Link"
 F 8 "311-1.69KFRCT-ND" H 1850 2500 60  0001 C CNN "Supplyer_Part_No"
-F 9 "311-1.69KFRTR-ND" H 1850 2500 60  0001 C CNN "Reel_Part_No"
-F 10 "5000" H 1850 2500 60  0001 C CNN "Parts_Per_Reel"
-F 11 ".1" H 1850 2500 60  0001 C CNN "Cost"
 	1    1850 2500
 	0    -1   1    0
@@
 F 7 "http://www.digikey.com/product-detail/en/yageo/RC1206JR-07300RL/311-300ERCT-ND/732222" H 1225 2500 60  0001 C CNN "Supplyer_Link"
 F 8 "311-300ERCT-ND" H 1225 2500 60  0001 C CNN "Supplyer_Part_No"
-F 9 "311-300ERTR-ND" H 1225 2500 60  0001 C CNN "Reel_Part_No"
-F 10 "5000" H 1225 2500 60  0001 C CNN "Parts_Per_Reel"
-F 11 ".1" H 1225 2500 60  0001 C CNN "Cost"
 	1    1225 2500
 	0    -1   1    0
@@
 F 7 "http://www.digikey.com/product-search/en?keywords=PS2801C-1-A" H 2775 2400 60  0001 C CNN "Supplyer_Link"
 F 8 "PS2801C-1-A-ND" H 2775 2400 60  0001 C CNN "Supplyer_Part_No"
-F 9 "PS2801C-1-F3-ATR-ND" H 2775 2400 60  0001 C CNN "Reel_Part_No"
-F 10 "3500" H 2775 2400 60  0001 C CNN "Parts_Per_Reel"
 	1    2775 2400
 	1    0    0    -1
@@
 F 7 "http://www.digikey.com/product-detail/en/yageo/RC1206FR-071KL/311-1.00KFRCT-ND/731334" H 3100 2725 60  0001 C CNN "Supplyer_Link"
 F 8 "311-1.00KFRCT-ND" H 3100 2725 60  0001 C CNN "Supplyer_Part_No"
-F 9 "311-1.00KFRTR-ND" H 3100 2725 60  0001 C CNN "Reel_Part_No"
-F 10 "5000" H 3100 2725 60  0001 C CNN "Parts_Per_Reel"
-F 11 ".1" H 3100 2725 60  0001 C CNN "Cost"
 	1    3100 2725
 	-1   0    0    -1
@@
 F 7 "http://www.digikey.com/product-search/en?keywords=CLM1B-AKW-CUAVB253CT-ND" H 3700 2550 60  0001 C CNN "Supplyer_Link"
 F 8 "CLM1B-AKW-CUAVB253CT-ND" H 3700 2550 60  0001 C CNN "Supplyer_Part_No"
-F 9 "CLM1B-AKW-CUAVB253TR-ND" H 3700 2550 60  0001 C CNN "Reel_Part_No"
-F 10 "2500" H 3700 2550 60  0001 C CNN "Parts_Per_Reel"
 	1    3700 2550
 	0    -1   -1   0
@@
 F 7 "http://www.digikey.com/product-detail/en/molex-llc/0015912060/WM17449-ND/614765" H 825 2350 60  0001 C CNN "Supplyer_Link"
 F 8 "WM17449-ND" H 825 2350 60  0001 C CNN "Supplyer_Part_No"
-F 9 "6600" H 825 2350 60  0001 C CNN "Parts_Per_Reel"
 	1    825  2350
 	-1   0    0    -1
@@
 F 7 "http://www.digikey.com/product-detail/en/3m/969102-0000-DA/3M9580-ND/2071621" H 1850 2750 60  0001 C CNN "Supplyer_Link"
 F 8 "3M9580-ND" H 1850 2750 60  0001 C CNN "Supplyer_Part_No"
-F 9 "None" H 1850 2750 60  0001 C CNN "Reel_Part_No"
-F 10 "None" H 1850 2750 60  0001 C CNN "Parts_Per_Reel"
 	1    1850 2750
 	-1   0    0    1
@@
 F 7 "-NA-" H 825 3025 60  0001 C CNN "Supplyer_Link"
 F 8 "-NA-" H 825 3025 60  0001 C CNN "Supplyer_Part_No"
-F 9 "-NA-" H 825 3025 60  0001 C CNN "Reel_Part_No"
-F 10 "-NA-" H 825 3025 60  0001 C CNN "Parts_Per_Reel"
 	1    825  3025
 	-1   0    0    -1
@@
 F 7 "http://www.digikey.com/product-detail/en/yageo/RC1206FR-07249RL/311-249FRCT-ND/731664" H 3100 3125 60  0001 C CNN "Supplyer_Link"
 F 8 "311-1.80KFRCT-ND" H 3100 3125 60  0001 C CNN "Supplyer_Part_No"
-F 9 "311-1.80FRTR-ND" H 3100 3125 60  0001 C CNN "Reel_Part_No"
-F 10 "5000" H 3100 3125 60  0001 C CNN "Parts_Per_Reel"
-F 11 ".1" H 3100 3125 60  0001 C CNN "Cost"
 	1    3100 3125
 	-1   0    0    -1
@@
 F 7 "http://www.digikey.com/products/en?keywords=311-3.60KFRCT-ND" H 3700 2250 60  0001 C CNN "Supplyer_Link"
 F 8 "311-3.60KFRCT-ND" H 3700 2250 60  0001 C CNN "Supplyer_Part_No"
-F 9 "311-3.60FRTR-ND" H 3700 2250 60  0001 C CNN "Reel_Part_No"
-F 10 "5000" H 3700 2250 60  0001 C CNN "Parts_Per_Reel"
 	1    3700 2250
 	-1   0    0    -1
@@
 F 7 "http://www.digikey.com/products/en?keywords=36-8197-ND" H 4800 2400 60  0001 C CNN "Supplyer_Link"
 F 8 "36-8197-ND" H 4800 2400 60  0001 C CNN "Supplyer_Part_No"
-F 9 "NA" H 4800 2400 60  0001 C CNN "Reel_Part_No"
-F 10 "NA" H 4800 2400 60  0001 C CNN "Parts_Per_Reel"
 	1    4800 2400
 	1    0    0    -1
@@
 F 3 "" H 2325 4575 60  0001 C CNN
 F 4 "Digi-Key" H 2325 4575 60  0001 C CNN "Supplyer"
-F 5 "Value" H 2325 4575 60  0001 C CNN "Parts_Per_Reel"
 	1    2325 4575
 	1    0    0    -1
@@
 F 7 "http://www.digikey.com/products/en?keywords=36-8197-ND" H 4800 2500 60  0001 C CNN "Supplyer_Link"
 F 8 "36-8197-ND" H 4800 2500 60  0001 C CNN "Supplyer_Part_No"
-F 9 "NA" H 4800 2500 60  0001 C CNN "Reel_Part_No"
-F 10 "NA" H 4800 2500 60  0001 C CNN "Parts_Per_Reel"
 	1    4800 2500
 	1    0    0    -1
@@
 F 7 "http://www.digikey.com/products/en?keywords=36-8197-ND" H 4800 2600 60  0001 C CNN "Supplyer_Link"
 F 8 "36-8197-ND" H 4800 2600 60  0001 C CNN "Supplyer_Part_No"
-F 9 "NA" H 4800 2600 60  0001 C CNN "Reel_Part_No"
-F 10 "NA" H 4800 2600 60  0001 C CNN "Parts_Per_Reel"
 	1    4800 2600
 	1    0    0    -1
@@
 F 7 "http://www.digikey.com/products/en?keywords=36-8197-ND" H 4800 2700 60  0001 C CNN "Supplyer_Link"
 F 8 "36-8197-ND" H 4800 2700 60  0001 C CNN "Supplyer_Part_No"
-F 9 "NA" H 4800 2700 60  0001 C CNN "Reel_Part_No"
-F 10 "NA" H 4800 2700 60  0001 C CNN "Parts_Per_Reel"
 	1    4800 2700
 	1    0    0    -1
